File: hardware/dev/1_1.kicad_sch (KiCad schematic)
At the start: 66 parts, among them P1 HDR-IDC-2_54-2X5P, U1 ZD24C02B-MAGMT, U10 RH-5015, U11 RH-5015, U12 RH-5015, U13 RH-5015, U14 RH-5015, U15 RH-5015, U16 RH-5015, U17 RH-5015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

Commit message: feat(hardware-dev): replace mode transistors with TPS2121 power mux
Parts:
- removed U26, U28: DMG2305UX-7, usb_sp_dev:SOT-23-3_L2.9-W1.3-P1.90-LS2.4-BR, symbol usb_sp_dev:DMG2305UX-7
- removed U34, U35, U36, U37: RH-5015, usb_sp_dev:SMD_RH-5015, symbol usb_sp_dev:RH-5015
- removed U5, U6: SN74LVC1G32DBVR, usb_sp:SOT-23-5_L3.0-W1.7-P0.95-LS2.8-BR, symbol usb_sp:SN74LVC1G32DBVR
- added C15: 100nF, Capacitor_SMD:C_0603_1608Metric, symbol Device:C
- added R13: 10kΩ, Resistor_SMD:R_0603_1608Metric, symbol Device:R
- added R14: 25.5kΩ, Resistor_SMD:R_0603_1608Metric, symbol Device:R
- added TP6, TP7, TP8: TestPoint, TestPoint:TestPoint_Pad_D1.0mm, symbol Connector:TestPoint
- added U5: SN74LVC1G08DBVR, usb_sp_dev:SOT-23-5_L3.0-W1.7-P0.95-LS2.8-BR, symbol usb_sp_dev:SN74LVC1G08DBVR
- added U6: TPS2121RUXR, usb_sp:VQFN-HR-12_L2.5-W2.0-P0.50-BL, symbol usb_sp:TPS2121RUXR
- R5, R7: footprint Resistor_SMD:R_0402_1005Metric -> Resistor_SMD:R_0603_1608Metric; LCSC Part Name 1kΩ ±1% 62.5mW 厚膜电阻 -> (none); Manufacturer UNI-ROYAL(厚声) -> (none); Manufacturer Part 0402WGF1001TCE -> (none); Supplier LCSC -> (none); Supplier Part C11702 -> (none)
- SMD-PAD-5x1, SMD-PAD-5x2, SMD-PAD-5x3, SMD-PAD-5x4, SMD-PAD-5x5, SMD-PAD-5x6: value ~ -> (none)
Connections:
- net USB_OUT_VBUS is gone; now on net VBUS: USB1.1 (VCC)
- net +3V3: now also R13.2, TP7.1, U5.5 (VCC)
- net GND: now also C15.2, R14.2, TP8.1, U5.3 (GND), U6.12 (GND), U6.3 (CP2), U6.4 (OV2), U6.5 (OV1), U6.6 (PR1), U6.9 (ST)
- net GPIO_RST_CH32: now also R13.1, U5.1 (A)
- net RST_CH32: now also U5.4 (Y)
- net RST_CH572: now also U5.2 (B)
- net USB_1_VBUS: now also U6.2 (IN2)
- net VBUS: now also U6.1 (OUT), U6.8 (OUT)
- net VBUS_FUSED: now also TP6.1
- new net: R14.1, U6.10 (ILM)
- new net: C15.1, U6.11 (SS)
- new net USB_2_VBUS: U6.7 (IN1)
Other:
- moved on the sheet: C10, C11, C12, C8, C9, D1, D2, TP1, TP2, TP3, TP4, TP5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
