File: hardware/prod/1_1.kicad_sch (KiCad schematic)
At the start: 40 parts, among them U1 CH32V203C8U6, U10 SN74LVC1G32DBVR, U2 ZD24C02B-MAGMT, U3 32.768kHz, U5 SD101CWS, U9 SN74LVC1G32DBVR, X1 8MHz

Commit message: feat(hardware-prod): replace mode transistors with TPS2121 power mux
Parts:
- removed TP1, TP2, TP3, TP4: TestPoint, TestPoint:TestPoint_Pad_D1.0mm, symbol Connector:TestPoint
- removed U10, U9: SN74LVC1G32DBVR, usb_sp_fp:SOT-23-5_L3.0-W1.7-P0.95-LS2.8-BR, symbol usb_sp:SN74LVC1G32DBVR
- added C15: 100nF, Capacitor_SMD:C_0402_1005Metric, symbol Device:C
- added R13: 10kΩ, Resistor_SMD:R_0402_1005Metric, symbol Device:R
- added R14: 25.5kΩ, Resistor_SMD:R_0402_1005Metric, symbol Device:R
- added RESET2: (no value), usb_sp_fp:SW-SMD_L3.9-W3.0-P4.45, symbol usb_sp:TS-1088-AR02016
- added U7: SN74LVC1G08DBVR, usb_sp_fp:SOT-23-5_L3.0-W1.7-P0.95-LS2.8-BR, symbol usb_sp_dev:SN74LVC1G08DBVR
- added U8: TPS2121RUXR, usb_sp_fp:VQFN-HR-12_L2.5-W2.0-P0.50-BL, symbol usb_sp:TPS2121RUXR
- C1, C13, C2: footprint Capacitor_SMD:C_0603_1608Metric -> Capacitor_SMD:C_0402_1005Metric; LCSC Part Name 10uF ±10% 10V -> CAP CER 10uF 10V X5R 0402; Manufacturer HRE(芯声) -> Samsung Electro-Mechanics; Manufacturer Part CGA0603X5R106K100JT -> CL05A106MP5NUNC; Supplier Part C6119842 -> C315248
- C6, C7, C8: footprint Capacitor_SMD:C_0603_1608Metric -> Capacitor_SMD:C_0402_1005Metric; LCSC Part Name 100nF ±10% 50V -> CAP CER 100nF 16V X7R 0402; Manufacturer HRE(芯声) -> YAGEO; Manufacturer Part CGA0603X7R104K500JT -> CC0402KRX7R7BB104; Supplier Part C6119867 -> C60474
- C9: footprint Capacitor_SMD:C_0603_1608Metric -> Capacitor_SMD:C_0402_1005Metric; LCSC Part Name 4.7uF ±10% 10V -> 4.7uF ±10% 10V Ceramic Capacitor X5R 0402; Manufacturer Part CL10A475KP8NNNC -> CL05A475KP5NRNC; Supplier Part C1705 -> C368809
- R10, R4, R5, R6, R9: footprint Resistor_SMD:R_0603_1608Metric -> Resistor_SMD:R_0402_1005Metric; LCSC Part Name 厚膜电阻 10kΩ ±5% 100mW -> RES 10kΩ ±1% 62.5mW 0402; Manufacturer Part RC0603JR-0710KL -> RC0402FR-0710KL; Supplier Part C99198 -> C60490
- RESET1, USER1: value ~ -> (none)
Connections:
- net +3V3: now also R13.2, RESET2.1, U7.5 (VCC); no longer R4.2, U1.44 (BOOT0)
- net GND: now also C15.2, R14.2, U7.3 (GND), U8.12 (GND), U8.3 (CP2), U8.4 (OV2), U8.5 (OV1), U8.6 (PR1), U8.9 (ST)
- net GPIO_RST_CH32: now also R13.1, U7.1 (A)
- net RST_CH32: now also U7.4 (Y)
- net RST_CH572: now also U7.2 (B)
- net VBUS: now also U8.1 (OUT), U8.8 (OUT); no longer USB1.1 (VCC)
- new net: R14.1, U8.10 (ILM)
- new net: C15.1, U8.11 (SS)
- new net BOOT_0: R4.2, RESET2.2, U1.44 (BOOT0)
- new net USB_1_VBUS: U8.2 (IN2), USB1.1 (VCC)
- new net USB_2_VBUS: U8.7 (IN1)
